File: pic_programmer/pic_programmer.kicad_pcb (KiCad board)
At the start: 2 copper layers, 160 x 99.1 mm, 63 parts, among them J1 DB9-FEMAL, P1 CONN_2, P101 CONN_1, P102 CONN_1, P103 CONN_1, P104 CONN_1, P105 CONN_1, P106 CONN_1, P2 SUPP28, P3 SUPP40, Q1 BC237, Q2 BC307, Q3 BC307, U1 24Cxx, U2 74HC125, U3 7805, U4 LT1373, U5 PIC_18_PINS, U6 PIC_8_PINS

Commit message: imported the netlist into pcb.
Parts:
- added P4: CONN_01X03, Sockets_MOLEX_KK-System:Socket_MOLEX-KK-RM2-54mm_Lock_3pin_straight, F.Cu at (227.3, 118.1)
- added P5: CONN_01X03, Sockets_MOLEX_KK-System:Socket_MOLEX-KK-RM3-96mm_Lock_3pin_straight, F.Cu at (209.6, 94.0)
- C9: value 22OnF -> 220nF
Connections:
- J1 pad 1: (no net) -> Net-(J1-Pad1)
- J1 pad 2: (no net) -> Net-(J1-Pad2)
- J1 pad 6: (no net) -> Net-(J1-Pad6)
- J1 pad 9: (no net) -> Net-(J1-Pad9)
- P101 pad 1: (no net) -> Net-(P101-Pad1)
- P102 pad 1: (no net) -> Net-(P102-Pad1)
- P103 pad 1: (no net) -> Net-(P103-Pad1)
- P104 pad 1: (no net) -> Net-(P104-Pad1)
- P105 pad 1: (no net) -> Net-(P105-Pad1)
- P106 pad 1: (no net) -> Net-(P106-Pad1)
- P2 pad 10: (no net) -> Net-(P2-Pad10)
- P2 pad 11: (no net) -> Net-(P2-Pad11)
- P2 pad 12: (no net) -> Net-(P2-Pad12)
- P2 pad 13: (no net) -> Net-(P2-Pad13)
- P2 pad 14: (no net) -> Net-(P2-Pad14)
- P2 pad 15: (no net) -> Net-(P2-Pad15)
- P2 pad 16: (no net) -> Net-(P2-Pad16)
- P2 pad 17: (no net) -> Net-(P2-Pad17)
- P2 pad 18: (no net) -> Net-(P2-Pad18)
- P2 pad 2: (no net) -> Net-(P2-Pad2)
- P2 pad 21: (no net) -> Net-(P2-Pad21)
- P2 pad 22: (no net) -> Net-(P2-Pad22)
- P2 pad 23: (no net) -> Net-(P2-Pad23)
- P2 pad 24: (no net) -> Net-(P2-Pad24)
- P2 pad 25: (no net) -> Net-(P2-Pad25)
- P2 pad 26: (no net) -> Net-(P2-Pad26)
- P2 pad 3: (no net) -> Net-(P2-Pad3)
- P2 pad 4: (no net) -> Net-(P2-Pad4)
- P2 pad 5: (no net) -> Net-(P2-Pad5)
- P2 pad 6: (no net) -> Net-(P2-Pad6)
- P2 pad 7: (no net) -> Net-(P2-Pad7)
- P2 pad 9: (no net) -> Net-(P2-Pad9)
- P3 pad 10: (no net) -> Net-(P3-Pad10)
- P3 pad 13: (no net) -> Net-(P3-Pad13)
- P3 pad 14: (no net) -> Net-(P3-Pad14)
- P3 pad 15: (no net) -> Net-(P3-Pad15)
- P3 pad 16: (no net) -> Net-(P3-Pad16)
- P3 pad 17: (no net) -> Net-(P3-Pad17)
- P3 pad 18: (no net) -> Net-(P3-Pad18)
- P3 pad 19: (no net) -> Net-(P3-Pad19)
- P3 pad 2: (no net) -> Net-(P3-Pad2)
- P3 pad 20: (no net) -> Net-(P3-Pad20)
- P3 pad 21: (no net) -> Net-(P3-Pad21)
- P3 pad 22: (no net) -> Net-(P3-Pad22)
- P3 pad 23: (no net) -> Net-(P3-Pad23)
- P3 pad 24: (no net) -> Net-(P3-Pad24)
- P3 pad 25: (no net) -> Net-(P3-Pad25)
- P3 pad 26: (no net) -> Net-(P3-Pad26)
- P3 pad 27: (no net) -> Net-(P3-Pad27)
- P3 pad 28: (no net) -> Net-(P3-Pad28)
- P3 pad 29: (no net) -> Net-(P3-Pad29)
- P3 pad 3: (no net) -> Net-(P3-Pad3)
- P3 pad 30: (no net) -> Net-(P3-Pad30)
- P3 pad 33: (no net) -> Net-(P3-Pad33)
- P3 pad 34: (no net) -> Net-(P3-Pad34)
- P3 pad 35: (no net) -> Net-(P3-Pad35)
- P3 pad 36: (no net) -> Net-(P3-Pad36)
- P3 pad 37: (no net) -> Net-(P3-Pad37)
- P3 pad 38: (no net) -> Net-(P3-Pad38)
- P3 pad 4: (no net) -> Net-(P3-Pad4)
- P3 pad 5: (no net) -> Net-(P3-Pad5)
- P3 pad 6: (no net) -> Net-(P3-Pad6)
- P3 pad 7: (no net) -> Net-(P3-Pad7)
- P3 pad 9: (no net) -> Net-(P3-Pad9)
- U1 pad 7: (no net) -> Net-(U1-Pad7)
- U4 pad 3: (no net) -> Net-(U4-Pad3)
- U4 pad 4: (no net) -> Net-(U4-Pad4)
- U5 pad 1: (no net) -> Net-(U5-Pad1)
- U5 pad 10: (no net) -> Net-(U5-Pad10)
- U5 pad 11: (no net) -> Net-(U5-Pad11)
- U5 pad 15: (no net) -> Net-(U5-Pad15)
- U5 pad 16: (no net) -> /pic_sockets/a3
- U5 pad 17: (no net) -> /pic_sockets/a2
- U5 pad 18: (no net) -> /pic_sockets/a1
- U5 pad 2: (no net) -> Net-(U5-Pad2)
- U5 pad 3: (no net) -> Net-(U5-Pad3)
- U5 pad 6: (no net) -> Net-(U5-Pad6)
- U5 pad 7: (no net) -> Net-(U5-Pad7)
- U5 pad 8: (no net) -> Net-(U5-Pad8)
- U5 pad 9: (no net) -> Net-(U5-Pad9)
- U6 pad 2: (no net) -> Net-(U6-Pad2)
- U6 pad 3: (no net) -> Net-(U6-Pad3)
- U6 pad 5: (no net) -> Net-(U6-Pad5)
